File: _restore_backup_2026-07-14T16-18-22-128/Tempmeasurementthingiemajig.kicad_sch (KiCad schematic)
At the start: 23 parts, among them J1 Conn_01x04_Socket, J2 Conn_01x05_Socket, J3 Conn_01x08_Pin, J4 Conn_01x08_Pin, J5 Conn_01x02_Pin, J6 Conn_01x02_Pin, U1 CMT2119A, U2 CH32V003FxPx, U3 SHT4x, Y1 26Mhz

Commit message: Worked on the pcb and exported it as gerbers+3d files
Parts:
- AE1: footprint Connector_PinHeader_2.54mm:PinHeader_1x01_P2.54mm_Vertical -> (none)
Changed lines of the file:
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@@
 			)
 		)
-		(property "Footprint" "Connector_PinHeader_2.54mm:PinHeader_1x01_P2.54mm_Vertical"
+		(property "Footprint" ""
 			(at 224.79 76.2 0)
 			(hide yes)
