File: _restore_backup_2026-07-14T16-18-22-128/old/Tempmeasurementthingiemajig.kicad_pcb (KiCad board)
At the start: 4 copper layers, 33.5 x 51.5 mm, 26 parts, among them J1 Conn_01x04_Socket, J2 Conn_01x05_Socket, J3 Conn_01x08_Pin, J4 Conn_01x08_Pin, J5 Conn_01x02_Pin, J6 Conn_01x02_Pin, U1 CMT2119A, U2 CH32V003FxPx, U3 SHT4x, Y1 26Mhz

Commit message: Worked on the pcb and exported it as gerbers+3d files
Parts:
- removed AE1: Antenna, Connector_PinHeader_2.54mm:PinHeader_1x01_P2.54mm_Vertical
- removed the G*** at (94.3, 113.6)
Routing:
- net Net-(AE1-A): track 2.37 -> 50.3 mm
Other:
- board text added: "868mHz RF"
- board text removed: "868MHz RF"
